File: Power.sch (EAGLE design)
At the start: 10 parts, among them IC1 LM340H-05

Commit message: final schematics
Parts:
- added F1: 3A, special:FUSE
- added J2: (no value), con-amp:MTA02-100
- added K1: AQG12105, relay:AQG12105
- added X1: 6ESRM-P, con-tycoelectronics:6ESRM-P
- added XL1: CFL-LAMP, ir:CFL-LAMP
- TR1: value (none) -> 120:9
Connections:
- new net N$10: F1.2, XL1.1, XL1.3
- new net N$11: F1.1, K1.DS2
- new net N$2: TR1.P1, X1.AC1, XL1.2, XL1.4
- new net N$6: K1.DS1, TR1.P2, X1.AC2
- new net N$7: J2.1, K1.K
- new net N$8: J2.2, K1.A
Other:
- note added: "- +"
- note added: "- Rly"
Changed lines of the file:
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@@
 </classes>
 <parts>
-<part name="TR1" library="trafo" deviceset="VP31" device=""/>
+<part name="TR1" library="trafo" deviceset="VP31" device="" value="120:9"/>
 <part name="D1" library="diode" deviceset="1N4004" device=""/>
 <part name="D2" library="diode" deviceset="1N4004" device=""/>
@@
 <part name="J1" library="con-amp" deviceset="MTA02-100" device=""/>
 <part name="IC1" library="linear" deviceset="LM340?-*" device="H" technology="05"/>
+<part name="K1" library="relay" deviceset="AQG*" device="" technology="12105"/>
+<part name="J2" library="con-amp" deviceset="MTA02-100" device=""/>
+<part name="F1" library="special" deviceset="FUSE" device="" value="3A"/>
+<part name="X1" library="con-tycoelectronics" deviceset="6ESRM-P" device=""/>
+<part name="XL1" library="ir" deviceset="CFL-LAMP" device=""/>
 </parts>
 <sheets>
 <sheet>
 <plain>
+<text x="125.73" y="52.578" size="1.778" layer="91" rot="R90">-   +</text>
+<text x="-27.94" y="19.558" size="1.778" layer="91" rot="R90">-  Rly</text>
 </plain>
 <instances>
@@
 <instance part="J1" gate="G$1" x="121.92" y="55.88" rot="R270"/>
 <instance part="IC1" gate="A" x="91.44" y="55.88"/>
+<instance part="K1" gate="A" x="-2.54" y="20.32"/>
+<instance part="J2" gate="G$1" x="-25.4" y="20.32" rot="R90"/>
+<instance part="F1" gate="G$1" x="22.86" y="17.78"/>
+<instance part="X1" gate="G$1" x="-15.24" y="53.34" rot="MR0"/>
+<instance part="XL1" gate="G$1" x="45.72" y="15.24"/>
 </instances>
 <busses>
@@
 </segment>
 </net>
+<net name="N$2" class="0">
+<segment>
+<pinref part="TR1" gate="1" pin="P1"/>
+<pinref part="X1" gate="G$1" pin="AC1"/>
+<wire x1="2.54" y1="58.42" x2="-2.54" y2="58.42" width="0.1524" layer="91"/>
+<junction x="-2.54" y="58.42"/>
+<wire x1="-2.54" y1="58.42" x2="-12.7" y2="58.42" width="0.1524" layer="91"/>
+<wire x1="-2.54" y1="58.42" x2="-2.54" y2="33.02" width="0.1524" layer="91"/>
+<wire x1="-2.54" y1="33.02" x2="55.88" y2="33.02" width="0.1524" layer="91"/>
+<pinref part="XL1" gate="G$1" pin="2"/>
+<wire x1="53.34" y1="10.16" x2="55.88" y2="10.16" width="0.1524" layer="91"/>
+<wire x1="55.88" y1="10.16" x2="55.88" y2="7.62" width="0.1524" layer="91"/>
+<pinref part="XL1" gate="G$1" pin="4"/>
+<wire x1="55.88" y1="7.62" x2="48.26" y2="7.62" width="0.1524" layer="91"/>
+<junction x="55.88" y="10.16"/>
+<wire x1="55.88" y1="33.02" x2="55.88" y2="10.16" width="0.1524" layer="91"/>
+</segment>
+</net>
+<net name="N$6" class="0">
+<segment>
+<pinref part="X1" gate="G$1" pin="AC2"/>
+<wire x1="-12.7" y1="48.26" x2="-7.62" y2="48.26" width="0.1524" layer="91"/>
+<wire x1="-7.62" y1="48.26" x2="-7.62" y2="45.72" width="0.1524" layer="91"/>
+<pinref part="TR1" gate="1" pin="P2"/>
+<wire x1="-7.62" y1="45.72" x2="2.54" y2="45.72" width="0.1524" layer="91"/>
+<wire x1="12.7" y1="30.48" x2="-7.62" y2="30.48" width="0.1524" layer="91"/>
+<wire x1="-7.62" y1="30.48" x2="-7.62" y2="45.72" width="0.1524" layer="91"/>
+<junction x="-7.62" y="45.72"/>
+<wire x1="12.7" y1="30.48" x2="12.7" y2="22.86" width="0.1524" layer="91"/>
+<pinref part="K1" gate="A" pin="DS1"/>
+<wire x1="12.7" y1="22.86" x2="7.62" y2="22.86" width="0.1524" layer="91"/>
+</segment>
+</net>
+<net name="N$7" class="0">
+<segment>
+<pinref part="K1" gate="A" pin="K"/>
+<pinref part="J2" gate="G$1" pin="1"/>
+<wire x1="-12.7" y1="17.78" x2="-17.78" y2="17.78" width="0.1524" layer="91"/>
+<wire x1="-17.78" y1="17.78" x2="-17.78" y2="20.32" width="0.1524" layer="91"/>
+<wire x1="-17.78" y1="20.32" x2="-22.86" y2="20.32" width="0.1524" layer="91"/>
+</segment>
+</net>
+<net name="N$8" class="0">
+<segment>
+<pinref part="K1" gate="A" pin="A"/>
+<pinref part="J2" gate="G$1" pin="2"/>
+<wire x1="-12.7" y1="22.86" x2="-22.86" y2="22.86" width="0.1524" layer="91"/>
+</segment>
+</net>
+<net name="N$10" class="0">
+<segment>
+<pinref part="XL1" gate="G$1" pin="1"/>
+<wire x1="38.1" y1="10.16" x2="35.56" y2="10.16" width="0.1524" layer="91"/>
+<pinref part="XL1" gate="G$1" pin="3"/>
+<wire x1="43.18" y1="7.62" x2="35.56" y2="7.62" width="0.1524" layer="91"/>
+<wire x1="35.56" y1="7.62" x2="35.56" y2="10.16" width="0.1524" layer="91"/>
+<pinref part="F1" gate="G$1" pin="2"/>
+<wire x1="27.94" y1="17.78" x2="35.56" y2="17.78" width="0.1524" layer="91"/>
+<wire x1="35.56" y1="17.78" x2="35.56" y2="10.16" width="0.1524" layer="91"/>
+<junction x="35.56" y="10.16"/>
+</segment>
+</net>
+<net name="N$11" class="0">
+<segment>
+<pinref part="F1" gate="G$1" pin="1"/>
+<pinref part="K1" gate="A" pin="DS2"/>
+<wire x1="15.24" y1="17.78" x2="7.62" y2="17.78" width="0.1524" layer="91"/>
+</segment>
+</net>

Commit message: reversed diodes D2 and D4 to correct orientation
Connections:
- net N$3: now also D2.A; no longer D2.C
- net N$4: now also D4.A; no longer D4.C
- net N$5: now also D2.C, D4.C; no longer D2.A, D4.A
Other:
- moved on the sheet: D2, D4
Changed lines of the file:
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@@
 <instance part="TR1" gate="1" x="7.62" y="53.34"/>
 <instance part="D1" gate="1" x="25.4" y="55.88"/>
-<instance part="D2" gate="1" x="50.8" y="55.88" rot="MR0"/>
+<instance part="D2" gate="1" x="43.18" y="55.88" rot="MR180"/>
 <instance part="D3" gate="1" x="25.4" y="48.26"/>
-<instance part="D4" gate="1" x="50.8" y="48.26" rot="MR0"/>
+<instance part="D4" gate="1" x="43.18" y="48.26" rot="MR180"/>
 <instance part="C1" gate="G$1" x="63.5" y="50.8"/>
 <instance part="C2" gate="G$1" x="76.2" y="50.8"/>
@@
 <segment>
 <pinref part="D1" gate="1" pin="C"/>
-<pinref part="D2" gate="1" pin="C"/>
 <wire x1="27.94" y1="55.88" x2="38.1" y2="55.88" width="0.1524" layer="91"/>
 <pinref part="TR1" gate="1" pin="S4"/>
-<wire x1="38.1" y1="55.88" x2="48.26" y2="55.88" width="0.1524" layer="91"/>
 <wire x1="15.24" y1="55.88" x2="17.78" y2="55.88" width="0.1524" layer="91"/>
 <wire x1="17.78" y1="55.88" x2="17.78" y2="60.96" width="0.1524" layer="91"/>
 <wire x1="17.78" y1="60.96" x2="38.1" y2="60.96" width="0.1524" layer="91"/>
 <wire x1="38.1" y1="60.96" x2="38.1" y2="55.88" width="0.1524" layer="91"/>
+<pinref part="D2" gate="1" pin="A"/>
+<wire x1="40.64" y1="55.88" x2="38.1" y2="55.88" width="0.1524" layer="91"/>
 <junction x="38.1" y="55.88"/>
 </segment>
@@
 <net name="N$4" class="0">
 <segment>
-<pinref part="D4" gate="1" pin="C"/>
 <pinref part="D3" gate="1" pin="C"/>
-<wire x1="48.26" y1="48.26" x2="38.1" y2="48.26" width="0.1524" layer="91"/>
 <pinref part="TR1" gate="1" pin="S3"/>
 <wire x1="38.1" y1="48.26" x2="27.94" y2="48.26" width="0.1524" layer="91"/>
@@
 <wire x1="17.78" y1="43.18" x2="38.1" y2="43.18" width="0.1524" layer="91"/>
 <wire x1="38.1" y1="43.18" x2="38.1" y2="48.26" width="0.1524" layer="91"/>
+<pinref part="D4" gate="1" pin="A"/>
+<wire x1="40.64" y1="48.26" x2="38.1" y2="48.26" width="0.1524" layer="91"/>
 <junction x="38.1" y="48.26"/>
 </segment>
@@
 <net name="N$5" class="0">
 <segment>
-<pinref part="D4" gate="1" pin="A"/>
-<wire x1="53.34" y1="48.26" x2="55.88" y2="48.26" width="0.1524" layer="91"/>
 <wire x1="55.88" y1="48.26" x2="55.88" y2="55.88" width="0.1524" layer="91"/>
-<pinref part="D2" gate="1" pin="A"/>
-<wire x1="55.88" y1="55.88" x2="53.34" y2="55.88" width="0.1524" layer="91"/>
 <pinref part="C1" gate="G$1" pin="1"/>
 <wire x1="63.5" y1="53.34" x2="63.5" y2="55.88" width="0.1524" layer="91"/>
@@
 <wire x1="76.2" y1="55.88" x2="63.5" y2="55.88" width="0.1524" layer="91"/>
 <wire x1="76.2" y1="53.34" x2="76.2" y2="55.88" width="0.1524" layer="91"/>
-<junction x="55.88" y="55.88"/>
 <junction x="76.2" y="55.88"/>
 <junction x="63.5" y="55.88"/>
+<pinref part="D2" gate="1" pin="C"/>
+<wire x1="45.72" y1="55.88" x2="55.88" y2="55.88" width="0.1524" layer="91"/>
+<pinref part="D4" gate="1" pin="C"/>
+<wire x1="45.72" y1="48.26" x2="55.88" y2="48.26" width="0.1524" layer="91"/>
+<junction x="55.88" y="55.88"/>
 </segment>
 </net>
